Commit message: update urdf

File: yumi_schunck_gym/assets/schunk_left_hand.urdf (robot description, URDF)
Before this commit: robot schunk_hand, 31 links, 30 joints
Joints:
- removed joint Part_hand
- added joint Part_Hand: type revolute, parent e1, child e2, origin xyz=-0.01840 0.006 0.0375 rpy=0 0 0, axis 0 0 -1, limit lower=0.0 upper=0.98786 effort=1000.0 velocity=1, mimic joint=Thumb_Opposition multiplier=1 offset=0

File: yumi_schunck_gym/assets/schunk_right_hand.urdf (robot description, URDF)
Before this commit: robot schunk_hand, 31 links, 30 joints
Joints:
- removed joint $j5
- added joint Part_Hand: type revolute, parent e1, child e2, origin xyz=0.01840 0.006 0.0375 rpy=0 0 0, axis 0 0 1, limit lower=0.0 upper=0.98786 effort=1000.0 velocity=1, mimic joint=Thumb_Opposition multiplier=1 offset=0

Commit message: Update schunk_left_hand.urdf

File: yumi_schunck_gym/assets/schunk_left_hand.urdf (robot description, URDF)
Before this commit: robot schunk_hand, 31 links, 30 joints
Links:
- removed link little_2
- removed link little_3
- removed link little_4
- removed link virtual_little_1
- added link pinky_2; collision mesh filename=package://meshes/f41.dae; visual mesh filename=package://meshes/f41.dae
- added link pinky_3; collision mesh filename=package://meshes/f42.dae; visual mesh filename=package://meshes/f42.dae
- added link pinky_4; collision mesh filename=package://meshes/f43.dae; visual mesh filename=package://meshes/f43.dae
- added link virtual_pinky_1; collision mesh filename=package://meshes/f40.dae; visual mesh filename=package://meshes/f40.dae
Joints:
- joint Pinky_3: child little_3 -> pinky_3; parent little_2 -> pinky_2
- joint Pinky_4: child little_4 -> pinky_4; parent little_3 -> pinky_3
- joint Pinky_Proximal: child little_2 -> pinky_2; parent virtual_little_1 -> virtual_pinky_1
- joint Pinky_Spread: child virtual_little_1 -> virtual_pinky_1
