Commit message: Update schunk_right_hand.urdf

File: yumi_schunck_gym/assets/schunk_right_hand.urdf (robot description, URDF)
Before this commit: robot schunk_hand, 31 links, 30 joints
Joints:
- removed joint Index_Finger_Proximal
- removed joint Middle_Finger_Proximal
- removed joint index_spread
- removed joint middle_spread_dummy
- added joint Index_Proximal: type revolute, parent virtual_l, child l, origin xyz=0 0 0 rpy=-1.5707 0 0, axis 0 0 1, limit lower=0.0 upper=0.79849 effort=1000.0 velocity=1
- added joint Index_Spread: type revolute, parent d2, child virtual_l, origin xyz=-0.025 0 0.110 rpy=0 -1.5707 1.5707, axis 0 0 1, limit lower=0.0 upper=0.28833 effort=1000.0 velocity=1, mimic joint=Finger_Spread multiplier=0.5 offset=0
- added joint Middle_Proximal: type revolute, parent virtual_k, child k, origin xyz=0 0 0 rpy=-1.5707 0 0, axis 0 0 1, limit lower=0.0 upper=0.79849 effort=1000.0 velocity=1
- added joint Middle_Spread_Dummy: type fixed, parent d, child virtual_k, origin xyz=0 0 0.110 rpy=0 -1.5707 1.5707

Commit message: Update schunk_right_hand.urdf

File: yumi_schunck_gym/assets/schunk_right_hand.urdf (robot description, URDF)
Before this commit: robot schunk_hand, 31 links, 30 joints
Joints:
- removed joint Finger_Spread
- removed joint Pinky
- removed joint Ring_Finger
- removed joint j12
- removed joint j13
- removed joint j16
- removed joint j17
- removed joint ring_spread
- added joint Pinky_3: type revolute, parent i, child m, origin xyz=0.04454 0 0 rpy=0 0 0, axis 0 0 1, limit lower=0 upper=1.334 effort=1000.0 velocity=1, mimic joint=Pinky_Proximal multiplier=1.35880 offset=0
- added joint Pinky_4: type revolute, parent m, child q, origin xyz=0.022 0 0 rpy=0 0 0, axis 0 0 1, limit lower=0 upper=1.3971 effort=1000.0 velocity=1, mimic joint=Pinky_Proximal multiplier=1.42307 offset=0
- added joint Pinky_Proximal: type revolute, parent virtual_i, child i, origin xyz=0 0 0 rpy=1.5707 0 0, axis 0 0 1, limit lower=0.0 upper=0.98175 effort=1000.0 velocity=1
- added joint Pinky_Spread: type revolute, parent e4, child virtual_i, origin xyz=0.025355 0 0.056 rpy=-1.5707 -1.5707 0, axis 0 0 1, limit lower=0.0 upper=0.5829 effort=1000.0 velocity=1
- added joint Ring_3: type revolute, parent j, child n, origin xyz=0.05004 0 0 rpy=0 0 0, axis 0 0 1, limit lower=0 upper=1.334 effort=1000.0 velocity=1, mimic joint=Ring_Proximal multiplier=1.3588 offset=0
- added joint Ring_4: type revolute, parent n, child r, origin xyz=0.032 0 0 rpy=0 0 0, axis 0 0 1, limit lower=0 upper=1.395 effort=1000.0 velocity=1, mimic joint=Ring_Proximal multiplier=1.42093 offset=0
- added joint Ring_Proximal: type revolute, parent virtual_j, child j, origin xyz=0 0 0 rpy=1.5707 0 0, axis 0 0 1, limit lower=0.0 upper=0.98175 effort=1000.0 velocity=1
- added joint Ring_Spread: type revolute, parent e5, child virtual_j, origin xyz=0.003855 0 0.0655 rpy=-1.5707 -1.5707 0, axis 0 0 1, limit lower=0.0 upper=0.28833 effort=1000.0 velocity=1, mimic joint=Pinky_Spread multiplier=0.5 offset=0
- joint Index_Spread: mimic joint=Finger_Spread multiplier=0.5 offset=0 -> joint=Pinky_Spread multiplier=0.5 offset=0

Commit message: Update schunk_right_hand.urdf

File: yumi_schunck_gym/assets/schunk_right_hand.urdf (robot description, URDF)
Before this commit: robot schunk_hand, 31 links, 30 joints
Links:
- removed link i
- removed link j
- removed link m
- removed link n
- removed link q
- removed link r
- removed link virtual_i
- removed link virtual_j
- added link pinky_2; collision mesh filename=package://meshes/f41.dae; visual mesh filename=package://meshes/f41.dae
- added link pinky_3; collision mesh filename=package://meshes/f42.dae; visual mesh filename=package://meshes/f42.dae
- added link pinky_4; collision mesh filename=package://meshes/f43.dae; visual mesh filename=package://meshes/f43.dae
- added link ring_2; collision mesh filename=package://meshes/f31.dae; visual mesh filename=package://meshes/f31.dae
- added link ring_3; collision mesh filename=package://meshes/f32.dae; visual mesh filename=package://meshes/f32.dae
- added link ring_4; collision mesh filename=package://meshes/f33.dae; visual mesh filename=package://meshes/f33.dae
- added link virtual_pinky_1; collision mesh filename=package://meshes/f40.dae; visual mesh filename=package://meshes/f40.dae
- added link virtual_ring_1; collision mesh filename=package://meshes/f30.dae; visual mesh filename=package://meshes/f30.dae
Joints:
- joint Pinky_3: child m -> pinky_3; parent i -> pinky_2
- joint Pinky_4: child q -> pinky_4; parent m -> pinky_3
- joint Pinky_Proximal: child i -> pinky_2; parent virtual_i -> virtual_pinky_1
- joint Pinky_Spread: child virtual_i -> virtual_pinky_1
- joint Ring_3: child n -> ring_3; parent j -> ring_2
- joint Ring_4: child r -> ring_4; parent n -> ring_3
- joint Ring_Proximal: child j -> ring_2; parent virtual_j -> virtual_ring_1
- joint Ring_Spread: child virtual_j -> virtual_ring_1

Commit message: Update schunk_right_hand.urdf

File: yumi_schunck_gym/assets/schunk_right_hand.urdf (robot description, URDF)
Before this commit: robot schunk_hand, 31 links, 30 joints
Links:
- removed link k
- removed link o
- removed link s
- removed link virtual_k
- added link middle_2; collision mesh filename=package://meshes/f21.dae; visual mesh filename=package://meshes/f21.dae
- added link middle_3; collision mesh filename=package://meshes/f22.dae; visual mesh filename=package://meshes/f22.dae
- added link middle_4; collision mesh filename=package://meshes/f23.dae; visual mesh filename=package://meshes/f23.dae
- added link virtual_middle_1; collision mesh filename=package://meshes/f20.dae; visual mesh filename=package://meshes/f20.dae
Joints:
- joint Middle_3: child o -> middle_3; parent k -> middle_2
- joint Middle_4: child s -> middle_4; parent o -> middle_3
- joint Middle_Proximal: child k -> middle_2; parent virtual_k -> virtual_middle_1
- joint Middle_Spread_Dummy: child virtual_k -> virtual_middle_1

Commit message: update urdf

File: yumi_schunck_gym/assets/schunk_right_hand.urdf (robot description, URDF)
Before this commit: robot schunk_hand, 31 links, 30 joints
Links:
- removed link l
- removed link p
- removed link t
- removed link virtual_l
- added link index_2; collision mesh filename=package://meshes/f11.dae; visual mesh filename=package://meshes/f11.dae
- added link index_3; collision mesh filename=package://meshes/f12.dae; visual mesh filename=package://meshes/f12.dae
- added link index_4; collision mesh filename=package://meshes/f13.dae; visual mesh filename=package://meshes/f13.dae
- added link virtual_index_1; collision mesh filename=package://meshes/f10.dae; visual mesh filename=package://meshes/f10.dae
Joints:
- joint Index_3: child p -> index_3; parent l -> index_2
- joint Index_4: child t -> index_4; parent p -> index_3
- joint Index_Proximal: child l -> index_2; parent virtual_l -> virtual_index_1
- joint Index_Spread: child virtual_l -> virtual_index_1

Commit message: Update schunk_right_hand.urdf

File: yumi_schunck_gym/assets/schunk_right_hand.urdf (robot description, URDF)
Before this commit: robot schunk_hand, 31 links, 30 joints
Links:
- removed link a
- removed link b
- removed link c
- removed link virtual_a
- removed link z
- added link thumb_1; collision mesh filename=package://meshes/d10.dae scale=1 1 1; visual mesh filename=package://meshes/d10.dae scale=1 1 1
- added link thumb_3; collision mesh filename=package://meshes/d11.dae scale=1 1 1; visual mesh filename=package://meshes/d11.dae scale=1 1 1
- added link thumb_4; collision mesh filename=package://meshes/d12.dae scale=1 1 1; visual mesh filename=package://meshes/d12.dae scale=1 1 1
- added link thumb_5; collision mesh filename=package://meshes/d13.dae scale=1 1 1; visual mesh filename=package://meshes/d13.dae scale=1 1 1
- added link thumb_virtual_2
Joints:
- joint Thumb_3: child b -> thumb_4; parent a -> thumb_3
- joint Thumb_4: child c -> thumb_5; parent b -> thumb_4
- joint Thumb_Flexion: child a -> thumb_3; parent virtual_a -> thumb_virtual_2
- joint Thumb_Helper: child virtual_a -> thumb_virtual_2; parent z -> thumb_1
- joint Thumb_Opposition: child z -> thumb_1
