Commit message: add schunk gym

File: yumi_gym/envs/assets/schunk_left_hand.urdf (robot description, URDF)
Before this commit: robot schunk_hand, 31 links, 30 joints
Links:
- removed link base_link
- removed link d
- removed link d2
- removed link e
- removed link e1
- removed link e2
- removed link e3
- removed link e4
- removed link e5
- removed link h
- removed link index_2
- removed link index_3
- removed link index_4
- removed link middle_2
- removed link middle_3
- removed link middle_4
- removed link pinky_2
- removed link pinky_3
- removed link pinky_4
- removed link thumb_1
- removed link thumb_3
- removed link thumb_4
- removed link thumb_5
- removed link thumb_virtual_2
- removed link virtual_index_1
- removed link virtual_middle_1
- removed link virtual_pinky_1
- added link Ld
- added link Ld2
- added link Le
- added link Le1; collision mesh filename=package://meshes/schunk_left/h10.dae scale=-1 1 1; visual mesh filename=package://meshes/schunk_left/h10.dae scale=-1 1 1
- added link Le2; collision mesh filename=package://meshes/schunk_left/h11.dae scale=-1 1 1; visual mesh filename=package://meshes/schunk_left/h11.dae scale=-1 1 1
- added link Le3
- added link Le4
- added link Le5
- added link Lh
- added link Lindex_2; collision mesh filename=package://meshes/schunk_left/f11.dae; visual mesh filename=package://meshes/schunk_left/f11.dae
- added link Lindex_3; collision mesh filename=package://meshes/schunk_left/f12.dae; visual mesh filename=package://meshes/schunk_left/f12.dae
- added link Lindex_4; collision mesh filename=package://meshes/schunk_left/f13.dae; visual mesh filename=package://meshes/schunk_left/f13.dae
- added link Lmiddle_2; collision mesh filename=package://meshes/schunk_left/f21.dae; visual mesh filename=package://meshes/schunk_left/f21.dae
- added link Lmiddle_3; collision mesh filename=package://meshes/schunk_left/f22.dae; visual mesh filename=package://meshes/schunk_left/f22.dae
- added link Lmiddle_4; collision mesh filename=package://meshes/schunk_left/f23.dae; visual mesh filename=package://meshes/schunk_left/f23.dae
- added link Lpinky_2; collision mesh filename=package://meshes/schunk_left/f41.dae; visual mesh filename=package://meshes/schunk_left/f41.dae
- added link Lpinky_3; collision mesh filename=package://meshes/schunk_left/f42.dae; visual mesh filename=package://meshes/schunk_left/f42.dae
- added link Lpinky_4; collision mesh filename=package://meshes/schunk_left/f43.dae; visual mesh filename=package://meshes/schunk_left/f43.dae
- added link Lthumb_1; collision mesh filename=package://meshes/schunk_left/d10.dae scale=1 -1 1; visual mesh filename=package://meshes/schunk_left/d10.dae scale=1 -1 1
- added link Lthumb_3; collision mesh filename=package://meshes/schunk_left/d11.dae scale=1 -1 -1; visual mesh filename=package://meshes/schunk_left/d11.dae scale=1 -1 -1
- added link Lthumb_4; collision mesh filename=package://meshes/schunk_left/d12.dae scale=1 -1 -1; visual mesh filename=package://meshes/schunk_left/d12.dae scale=1 -1 -1
- added link Lthumb_5; collision mesh filename=package://meshes/schunk_left/d13.dae scale=1 -1 -1; visual mesh filename=package://meshes/schunk_left/d13.dae scale=1 -1 -1
- added link Lthumb_virtual_2
- added link Lvirtual_index_1; collision mesh filename=package://meshes/schunk_left/f10.dae; visual mesh filename=package://meshes/schunk_left/f10.dae
- added link Lvirtual_middle_1; collision mesh filename=package://meshes/schunk_left/f20.dae; visual mesh filename=package://meshes/schunk_left/f20.dae
- added link Lvirtual_pinky_1; collision mesh filename=package://meshes/schunk_left/f40.dae; visual mesh filename=package://meshes/schunk_left/f40.dae
- added link left_hand_base; collision mesh filename=package://meshes/schunk_left/base10.dae; visual mesh filename=package://meshes/schunk_left/base10.dae
- link ring_2: geometry collision mesh filename=package://meshes/schunk_left/f31.dae; visual mesh filename=package://meshes/schunk_left/f31.dae
- link ring_3: geometry collision mesh filename=package://meshes/schunk_left/f32.dae; visual mesh filename=package://meshes/schunk_left/f32.dae
- link ring_4: geometry collision mesh filename=package://meshes/schunk_left/f33.dae; visual mesh filename=package://meshes/schunk_left/f33.dae
- link virtual_ring_1: geometry collision mesh filename=package://meshes/schunk_left/f30.dae; visual mesh filename=package://meshes/schunk_left/f30.dae
Joints:
- removed joint Index_3
- removed joint Index_4
- removed joint Index_Proximal
- removed joint Index_Spread
- removed joint Middle_3
- removed joint Middle_4
- removed joint Middle_Proximal
- removed joint Middle_Spread_Dummy
- removed joint Part_Hand
- removed joint Pinky_3
- removed joint Pinky_4
- removed joint Pinky_Proximal
- removed joint Pinky_Spread
- removed joint Ring_3
- removed joint Ring_4
- removed joint Ring_Proximal
- removed joint Ring_Spread
- removed joint Thumb_3
- removed joint Thumb_4
- removed joint Thumb_Flexion
- removed joint Thumb_Helper
- removed joint Thumb_Opposition
- removed joint f1
- removed joint f2
- removed joint f3
- removed joint f4
- removed joint f5
- removed joint f6
- removed joint f7
- removed joint f8
- added joint LIndex_3: type revolute, parent Lindex_2, child Lindex_3, origin xyz=0.04804 0 0 rpy=0 0 0, axis 0 0 1, limit lower=0 upper=1.334 effort=1000.0 velocity=1
- added joint LIndex_4: type revolute, parent Lindex_3, child Lindex_4, origin xyz=0.026 0 0 rpy=0 0 0, axis 0 0 1, limit lower=0 upper=1.394 effort=1000.0 velocity=1, mimic joint=LIndex_3 multiplier=1.0450 offset=0
- added joint LIndex_Proximal: type revolute, parent Lvirtual_index_1, child Lindex_2, origin xyz=0 0 0 rpy=-1.5707 0 0, axis 0 0 1, limit lower=0.0 upper=0.79849 effort=1000.0 velocity=1
- added joint LIndex_Spread: type revolute, parent Ld2, child Lvirtual_index_1, origin xyz=0.025 0 0.110 rpy=0 -1.5707 1.5707, axis 0 0 -1, limit lower=0.0 upper=0.28833 effort=1000.0 velocity=1, mimic joint=LPinky_Spread multiplier=0.5 offset=0
- added joint LMiddle_3: type revolute, parent Lmiddle_2, child Lmiddle_3, origin xyz=0.05004 0 0 rpy=0 0 0, axis 0 0 1, limit lower=0 upper=1.334 effort=1000.0 velocity=1
- added joint LMiddle_4: type revolute, parent Lmiddle_3, child Lmiddle_4, origin xyz=0.032 0 0 rpy=0 0 0, axis 0 0 1, limit lower=0 upper=1.334 effort=1000.0 velocity=1, mimic joint=LMiddle_3 multiplier=1.0454 offset=0
- added joint LMiddle_Proximal: type revolute, parent Lvirtual_middle_1, child Lmiddle_2, origin xyz=0 0 0 rpy=-1.5707 0 0, axis 0 0 1, limit lower=0.0 upper=0.79849 effort=1000.0 velocity=1
- added joint LMiddle_Spread_Dummy: type fixed, parent Ld, child Lvirtual_middle_1, origin xyz=0 0 0.110 rpy=0 -1.5707 1.5707
- added joint LPart_Hand: type revolute, parent Le1, child Le2, origin xyz=-0.01840 0.006 0.0375 rpy=0 0 0, axis 0 0 -1, limit lower=0.0 upper=0.98786 effort=1000.0 velocity=1, mimic joint=LThumb_Opposition multiplier=1 offset=0
- added joint LPinky_3: type revolute, parent Lpinky_2, child Lpinky_3, origin xyz=0.04454 0 0 rpy=0 0 0, axis 0 0 1, limit lower=0 upper=1.334 effort=1000.0 velocity=1, mimic joint=LPinky_Proximal multiplier=1.35880 offset=0
- added joint LPinky_4: type revolute, parent Lpinky_3, child Lpinky_4, origin xyz=0.022 0 0 rpy=0 0 0, axis 0 0 1, limit lower=0 upper=1.3971 effort=1000.0 velocity=1, mimic joint=LPinky_Proximal multiplier=1.42307 offset=0
- added joint LPinky_Proximal: type revolute, parent Lvirtual_pinky_1, child Lpinky_2, origin xyz=0 0 0 rpy=1.5707 0 0, axis 0 0 1, limit lower=0.0 upper=0.98175 effort=1000.0 velocity=1
- added joint LPinky_Spread: type revolute, parent Le4, child Lvirtual_pinky_1, origin xyz=-0.025355 0 0.056 rpy=-1.5707 -1.5707 0, axis 0 0 -1, limit lower=0.0 upper=0.5829 effort=1000.0 velocity=1
- added joint LRing_3: type revolute, parent ring_2, child ring_3, origin xyz=0.05004 0 0 rpy=0 0 0, axis 0 0 1, limit lower=0 upper=1.334 effort=1000.0 velocity=1, mimic joint=LRing_Proximal multiplier=1.3588 offset=0
- added joint LRing_4: type revolute, parent ring_3, child ring_4, origin xyz=0.032 0 0 rpy=0 0 0, axis 0 0 1, limit lower=0 upper=1.395 effort=1000.0 velocity=1, mimic joint=LRing_Proximal multiplier=1.42093 offset=0
- added joint LRing_Proximal: type revolute, parent virtual_ring_1, child ring_2, origin xyz=0 0 0 rpy=1.5707 0 0, axis 0 0 1, limit lower=0.0 upper=0.98175 effort=1000.0 velocity=1
- added joint LRing_Spread: type revolute, parent Le5, child virtual_ring_1, origin xyz=-0.003855 0 0.0655 rpy=-1.5707 -1.5707 0, axis 0 0 -1, limit lower=0.0 upper=0.28833 effort=1000.0 velocity=1, mimic joint=LPinky_Spread multiplier=0.5 offset=0
- added joint LThumb_3: type revolute, parent Lthumb_3, child Lthumb_4, origin xyz=0.0485 0 0 rpy=0 0 0, axis 0 0 -1, limit lower=0.0 upper=0.98506 effort=1000.0 velocity=1, mimic joint=LThumb_Flexion multiplier=1.01511 offset=0
- added joint LThumb_4: type revolute, parent Lthumb_4, child Lthumb_5, origin xyz=0.030 0 0 rpy=0 0 0, axis 0 0 -1, limit lower=0.0 upper=1.406 effort=1000.0 velocity=1, mimic joint=LThumb_Flexion multiplier=1.44889 offset=0
- added joint LThumb_Flexion: type revolute, parent Lthumb_virtual_2, child Lthumb_3, origin xyz=0 0 0 rpy=0 0 0.9704, axis 0 0 -1, limit lower=0.0 upper=0.9704 effort=1000.0 velocity=1
- added joint LThumb_Helper: type fixed, parent Lthumb_1, child Lthumb_virtual_2, origin xyz=0 0 0.04596 rpy=0 -1.5707 3.1416
- added joint LThumb_Opposition: type revolute, parent Le1, child Lthumb_1, origin xyz=0.01690 0.02626 0 rpy=0 0.2618 1.571, axis 0 0 1, limit lower=0.0 upper=0.9879 effort=1000.0 velocity=1
- added joint Lf1: type fixed, parent Le1, child Ld, origin xyz=0 0 0 rpy=0 0 0
- added joint Lf2: type fixed, parent Ld, child Lh, origin xyz=0 0 0 rpy=0 0 0
- added joint Lf3: type fixed, parent Lh, child Ld2, origin xyz=0 0 0 rpy=0 0 0
- added joint Lf4: type fixed, parent left_hand_base, child Le1, origin xyz=0 -0.01313 0 rpy=0 0 0
- added joint Lf5: type fixed, parent Le2, child Le3, origin xyz=0 -0.0060 0 rpy=0 0 0
- added joint Lf6: type fixed, parent Le3, child Le, origin xyz=0 0 0 rpy=0 0 0
- added joint Lf7: type fixed, parent Le, child Le4, origin xyz=0 0 0 rpy=0 0 0
- added joint Lf8: type fixed, parent Le, child Le5, origin xyz=0 0 0 rpy=0 0 0

File: yumi_gym/envs/assets/schunk_right_hand.urdf (robot description, URDF)
Before this commit: robot schunk_hand, 31 links, 30 joints
Links:
- removed link base_link
- removed link d
- removed link d2
- removed link e
- removed link e1
- removed link e2
- removed link e3
- removed link e4
- removed link e5
- removed link h
- removed link index_2
- removed link index_3
- removed link index_4
- removed link middle_2
- removed link middle_3
- removed link middle_4
- removed link pinky_2
- removed link pinky_3
- removed link pinky_4
- removed link ring_2
- removed link ring_3
- removed link ring_4
- removed link thumb_1
- removed link thumb_3
- removed link thumb_4
- removed link thumb_5
- removed link thumb_virtual_2
- removed link virtual_index_1
- removed link virtual_middle_1
- removed link virtual_pinky_1
- removed link virtual_ring_1
- added link Rd
- added link Rd2
- added link Re
- added link Re1; collision mesh filename=package://meshes/schunk_right/h10.dae scale=1 1 1; visual mesh filename=package://meshes/schunk_right/h10.dae scale=1 1 1
- added link Re2; collision mesh filename=package://meshes/schunk_right/h11.dae scale=1 1 1; visual mesh filename=package://meshes/schunk_right/h11.dae scale=1 1 1
- added link Re3
- added link Re4
- added link Re5
- added link Rh
- added link Rindex_2; collision mesh filename=package://meshes/schunk_right/f11.dae; visual mesh filename=package://meshes/schunk_right/f11.dae
- added link Rindex_3; collision mesh filename=package://meshes/schunk_right/f12.dae; visual mesh filename=package://meshes/schunk_right/f12.dae
- added link Rindex_4; collision mesh filename=package://meshes/schunk_right/f13.dae; visual mesh filename=package://meshes/schunk_right/f13.dae
- added link Rmiddle_2; collision mesh filename=package://meshes/schunk_right/f21.dae; visual mesh filename=package://meshes/schunk_right/f21.dae
- added link Rmiddle_3; collision mesh filename=package://meshes/schunk_right/f22.dae; visual mesh filename=package://meshes/schunk_right/f22.dae
- added link Rmiddle_4; collision mesh filename=package://meshes/schunk_right/f23.dae; visual mesh filename=package://meshes/schunk_right/f23.dae
- added link Rpinky_2; collision mesh filename=package://meshes/schunk_right/f41.dae; visual mesh filename=package://meshes/schunk_right/f41.dae
- added link Rpinky_3; collision mesh filename=package://meshes/schunk_right/f42.dae; visual mesh filename=package://meshes/schunk_right/f42.dae
- added link Rpinky_4; collision mesh filename=package://meshes/schunk_right/f43.dae; visual mesh filename=package://meshes/schunk_right/f43.dae
- added link Rring_2; collision mesh filename=package://meshes/schunk_right/f31.dae; visual mesh filename=package://meshes/schunk_right/f31.dae
- added link Rring_3; collision mesh filename=package://meshes/schunk_right/f32.dae; visual mesh filename=package://meshes/schunk_right/f32.dae
- added link Rring_4; collision mesh filename=package://meshes/schunk_right/f33.dae; visual mesh filename=package://meshes/schunk_right/f33.dae
- added link Rthumb_1; collision mesh filename=package://meshes/schunk_right/d10.dae scale=1 1 1; visual mesh filename=package://meshes/schunk_right/d10.dae scale=1 1 1
- added link Rthumb_3; collision mesh filename=package://meshes/schunk_right/d11.dae scale=1 1 1; visual mesh filename=package://meshes/schunk_right/d11.dae scale=1 1 1
- added link Rthumb_4; collision mesh filename=package://meshes/schunk_right/d12.dae scale=1 1 1; visual mesh filename=package://meshes/schunk_right/d12.dae scale=1 1 1
- added link Rthumb_5; collision mesh filename=package://meshes/schunk_right/d13.dae scale=1 1 1; visual mesh filename=package://meshes/schunk_right/d13.dae scale=1 1 1
- added link Rthumb_virtual_2
- added link Rvirtual_index_1; collision mesh filename=package://meshes/schunk_right/f10.dae; visual mesh filename=package://meshes/schunk_right/f10.dae
- added link Rvirtual_middle_1; collision mesh filename=package://meshes/schunk_right/f20.dae; visual mesh filename=package://meshes/schunk_right/f20.dae
- added link Rvirtual_pinky_1; collision mesh filename=package://meshes/schunk_right/f40.dae; visual mesh filename=package://meshes/schunk_right/f40.dae
- added link Rvirtual_ring_1; collision mesh filename=package://meshes/schunk_right/f30.dae; visual mesh filename=package://meshes/schunk_right/f30.dae
- added link right_hand_base; collision mesh filename=package://meshes/schunk_right/base10.dae; visual mesh filename=package://meshes/schunk_right/base10.dae
Joints:
- removed joint Index_3
- removed joint Index_4
- removed joint Index_Proximal
- removed joint Index_Spread
- removed joint Middle_3
- removed joint Middle_4
- removed joint Middle_Proximal
- removed joint Middle_Spread_Dummy
- removed joint Part_Hand
- removed joint Pinky_3
- removed joint Pinky_4
- removed joint Pinky_Proximal
- removed joint Pinky_Spread
- removed joint Ring_3
- removed joint Ring_4
- removed joint Ring_Proximal
- removed joint Ring_Spread
- removed joint Thumb_3
- removed joint Thumb_4
- removed joint Thumb_Flexion
- removed joint Thumb_Helper
- removed joint Thumb_Opposition
- removed joint f1
- removed joint f2
- removed joint f3
- removed joint f4
- removed joint f5
- removed joint f6
- removed joint f7
- removed joint f8
- added joint RIndex_3: type revolute, parent Rindex_2, child Rindex_3, origin xyz=0.04804 0 0 rpy=0 0 0, axis 0 0 1, limit lower=0 upper=1.334 effort=1000.0 velocity=1
- added joint RIndex_4: type revolute, parent Rindex_3, child Rindex_4, origin xyz=0.026 0 0 rpy=0 0 0, axis 0 0 1, limit lower=0 upper=1.394 effort=1000.0 velocity=1, mimic joint=RIndex_3 multiplier=1.0450 offset=0
- added joint RIndex_Proximal: type revolute, parent Rvirtual_index_1, child Rindex_2, origin xyz=0 0 0 rpy=-1.5707 0 0, axis 0 0 1, limit lower=0.0 upper=0.79849 effort=1000.0 velocity=1
- added joint RIndex_Spread: type revolute, parent Rd2, child Rvirtual_index_1, origin xyz=-0.025 0 0.110 rpy=0 -1.5707 1.5707, axis 0 0 1, limit lower=0.0 upper=0.28833 effort=1000.0 velocity=1, mimic joint=RPinky_Spread multiplier=0.5 offset=0
- added joint RMiddle_3: type revolute, parent Rmiddle_2, child Rmiddle_3, origin xyz=0.05004 0 0 rpy=0 0 0, axis 0 0 1, limit lower=0 upper=1.334 effort=1000.0 velocity=1
- added joint RMiddle_4: type revolute, parent Rmiddle_3, child Rmiddle_4, origin xyz=0.032 0 0 rpy=0 0 0, axis 0 0 1, limit lower=0 upper=1.334 effort=1000.0 velocity=1, mimic joint=RMiddle_3 multiplier=1.0454 offset=0
- added joint RMiddle_Proximal: type revolute, parent Rvirtual_middle_1, child Rmiddle_2, origin xyz=0 0 0 rpy=-1.5707 0 0, axis 0 0 1, limit lower=0.0 upper=0.79849 effort=1000.0 velocity=1
- added joint RMiddle_Spread_Dummy: type fixed, parent Rd, child Rvirtual_middle_1, origin xyz=0 0 0.110 rpy=0 -1.5707 1.5707
- added joint RPart_Hand: type revolute, parent Re1, child Re2, origin xyz=0.01840 0.006 0.0375 rpy=0 0 0, axis 0 0 1, limit lower=0.0 upper=0.98786 effort=1000.0 velocity=1, mimic joint=RThumb_Opposition multiplier=1 offset=0
- added joint RPinky_3: type revolute, parent Rpinky_2, child Rpinky_3, origin xyz=0.04454 0 0 rpy=0 0 0, axis 0 0 1, limit lower=0 upper=1.334 effort=1000.0 velocity=1, mimic joint=RPinky_Proximal multiplier=1.35880 offset=0
- added joint RPinky_4: type revolute, parent Rpinky_3, child Rpinky_4, origin xyz=0.022 0 0 rpy=0 0 0, axis 0 0 1, limit lower=0 upper=1.3971 effort=1000.0 velocity=1, mimic joint=RPinky_Proximal multiplier=1.42307 offset=0
- added joint RPinky_Proximal: type revolute, parent Rvirtual_pinky_1, child Rpinky_2, origin xyz=0 0 0 rpy=1.5707 0 0, axis 0 0 1, limit lower=0.0 upper=0.98175 effort=1000.0 velocity=1
- added joint RPinky_Spread: type revolute, parent Re4, child Rvirtual_pinky_1, origin xyz=0.025355 0 0.056 rpy=-1.5707 -1.5707 0, axis 0 0 1, limit lower=0.0 upper=0.5829 effort=1000.0 velocity=1
- added joint RRing_3: type revolute, parent Rring_2, child Rring_3, origin xyz=0.05004 0 0 rpy=0 0 0, axis 0 0 1, limit lower=0 upper=1.334 effort=1000.0 velocity=1, mimic joint=RRing_Proximal multiplier=1.3588 offset=0
- added joint RRing_4: type revolute, parent Rring_3, child Rring_4, origin xyz=0.032 0 0 rpy=0 0 0, axis 0 0 1, limit lower=0 upper=1.395 effort=1000.0 velocity=1, mimic joint=RRing_Proximal multiplier=1.42093 offset=0
- added joint RRing_Proximal: type revolute, parent Rvirtual_ring_1, child Rring_2, origin xyz=0 0 0 rpy=1.5707 0 0, axis 0 0 1, limit lower=0.0 upper=0.98175 effort=1000.0 velocity=1
- added joint RRing_Spread: type revolute, parent Re5, child Rvirtual_ring_1, origin xyz=0.003855 0 0.0655 rpy=-1.5707 -1.5707 0, axis 0 0 1, limit lower=0.0 upper=0.28833 effort=1000.0 velocity=1, mimic joint=RPinky_Spread multiplier=0.5 offset=0
- added joint RThumb_3: type revolute, parent Rthumb_3, child Rthumb_4, origin xyz=0.0485 0 0 rpy=0 0 0, axis 0 0 1, limit lower=0.0 upper=0.98506 effort=1000.0 velocity=1, mimic joint=RThumb_Flexion multiplier=1.01511 offset=0
- added joint RThumb_4: type revolute, parent Rthumb_4, child Rthumb_5, origin xyz=0.030 0 0 rpy=0 0 0, axis 0 0 1, limit lower=0.0 upper=1.406 effort=1000.0 velocity=1, mimic joint=RThumb_Flexion multiplier=1.44889 offset=0
- added joint RThumb_Flexion: type revolute, parent Rthumb_virtual_2, child Rthumb_3, origin xyz=0 0 0 rpy=0 0 -0.9704, axis 0 0 1, limit lower=0.0 upper=0.9704 effort=1000.0 velocity=1
- added joint RThumb_Helper: type fixed, parent Rthumb_1, child Rthumb_virtual_2, origin xyz=0 0 0.04596 rpy=0 -1.5707 3.1416
- added joint RThumb_Opposition: type revolute, parent Re1, child Rthumb_1, origin xyz=-0.01690 0.02626 0 rpy=0 0.2618 1.571, axis 0 0 -1, limit lower=0.0 upper=0.9879 effort=1000.0 velocity=1
- added joint Rf1: type fixed, parent Re1, child Rd, origin xyz=0 0 0 rpy=0 0 0
- added joint Rf2: type fixed, parent Rd, child Rh, origin xyz=0 0 0 rpy=0 0 0
- added joint Rf3: type fixed, parent Rh, child Rd2, origin xyz=0 0 0 rpy=0 0 0
- added joint Rf4: type fixed, parent right_hand_base, child Re1, origin xyz=0 -0.01313 0 rpy=0 0 0
- added joint Rf5: type fixed, parent Re2, child Re3, origin xyz=0 -0.0060 0 rpy=0 0 0
- added joint Rf6: type fixed, parent Re3, child Re, origin xyz=0 0 0 rpy=0 0 0
- added joint Rf7: type fixed, parent Re, child Re4, origin xyz=0 0 0 rpy=0 0 0
- added joint Rf8: type fixed, parent Re, child Re5, origin xyz=0 0 0 rpy=0 0 0
