Commit message: add schunk gym

File: yumi_gym/envs/assets/yumi_with_inspire_hands.urdf (robot description, URDF)
Before this commit: robot yumi, 45 links, 44 joints
Links:
- link Link1: geometry collision mesh filename=package://meshes/inspire_right/Link1.STL; visual mesh filename=package://meshes/inspire_right/Link1.STL
- link Link11: geometry collision mesh filename=package://meshes/inspire_right/Link11.STL; visual mesh filename=package://meshes/inspire_right/Link11.STL
- link Link111: geometry collision mesh filename=package://meshes/inspire_right/Link111.STL; visual mesh filename=package://meshes/inspire_right/Link111.STL
- link Link2: geometry collision mesh filename=package://meshes/inspire_right/Link2.STL; visual mesh filename=package://meshes/inspire_right/Link2.STL
- link Link22: geometry collision mesh filename=package://meshes/inspire_right/Link22.STL; visual mesh filename=package://meshes/inspire_right/Link22.STL
- link Link3: geometry collision mesh filename=package://meshes/inspire_right/Link3.STL; visual mesh filename=package://meshes/inspire_right/Link3.STL
- link Link33: geometry collision mesh filename=package://meshes/inspire_right/Link33.STL; visual mesh filename=package://meshes/inspire_right/Link33.STL
- link Link4: geometry collision mesh filename=package://meshes/inspire_right/Link4.STL; visual mesh filename=package://meshes/inspire_right/Link4.STL
- link Link44: geometry collision mesh filename=package://meshes/inspire_right/Link44.STL; visual mesh filename=package://meshes/inspire_right/Link44.STL
- link Link5: geometry collision mesh filename=package://meshes/inspire_right/Link5.STL; visual mesh filename=package://meshes/inspire_right/Link5.STL
- link Link51: geometry collision mesh filename=package://meshes/inspire_right/Link51.STL; visual mesh filename=package://meshes/inspire_right/Link51.STL
- link Link52: geometry collision mesh filename=package://meshes/inspire_right/Link52.STL; visual mesh filename=package://meshes/inspire_right/Link52.STL
- link Link53: geometry collision mesh filename=package://meshes/inspire_right/Link53.STL; visual mesh filename=package://meshes/inspire_right/Link53.STL
- link link1: geometry collision mesh filename=package://meshes/inspire_left/link1.STL; visual mesh filename=package://meshes/inspire_left/link1.STL
- link link11: geometry collision mesh filename=package://meshes/inspire_left/link11.STL; visual mesh filename=package://meshes/inspire_left/link11.STL
- link link111: geometry collision mesh filename=package://meshes/inspire_left/link111.STL; visual mesh filename=package://meshes/inspire_left/link111.STL
- link link2: geometry collision mesh filename=package://meshes/inspire_left/link2.STL; visual mesh filename=package://meshes/inspire_left/link2.STL
- link link22: geometry collision mesh filename=package://meshes/inspire_left/link22.STL; visual mesh filename=package://meshes/inspire_left/link22.STL
- link link3: geometry collision mesh filename=package://meshes/inspire_left/link3.STL; visual mesh filename=package://meshes/inspire_left/link3.STL
- link link33: geometry collision mesh filename=package://meshes/inspire_left/link33.STL; visual mesh filename=package://meshes/inspire_left/link33.STL
- link link4: geometry collision mesh filename=package://meshes/inspire_left/link4.STL; visual mesh filename=package://meshes/inspire_left/link4.STL
- link link44: geometry collision mesh filename=package://meshes/inspire_left/link44.STL; visual mesh filename=package://meshes/inspire_left/link44.STL
- link link5: geometry collision mesh filename=package://meshes/inspire_left/link5.STL; visual mesh filename=package://meshes/inspire_left/link5.STL
- link link51: geometry collision mesh filename=package://meshes/inspire_left/link51.STL; visual mesh filename=package://meshes/inspire_left/link51.STL
- link link52: geometry collision mesh filename=package://meshes/inspire_left/link52.STL; visual mesh filename=package://meshes/inspire_left/link52.STL
- link link53: geometry collision mesh filename=package://meshes/inspire_left/link53.STL; visual mesh filename=package://meshes/inspire_left/link53.STL

Commit message: .dae to .stl and add .xml

File: yumi_gym/envs/assets/schunk_left_hand.urdf (robot description, URDF)
Before this commit: robot left_schunk_hand, 31 links, 30 joints
Links:
- link Le1: geometry collision mesh filename=package://meshes/schunk_left/h10.stl scale=-1 1 1; visual mesh filename=package://meshes/schunk_left/h10.stl scale=-1 1 1
- link Le2: geometry collision mesh filename=package://meshes/schunk_left/h11.stl scale=-1 1 1; visual mesh filename=package://meshes/schunk_left/h11.stl scale=-1 1 1
- link Lindex_2: geometry collision mesh filename=package://meshes/schunk_left/f11.stl; visual mesh filename=package://meshes/schunk_left/f11.stl
- link Lindex_3: geometry collision mesh filename=package://meshes/schunk_left/f12.stl; visual mesh filename=package://meshes/schunk_left/f12.stl
- link Lindex_4: geometry collision mesh filename=package://meshes/schunk_left/f13.stl; visual mesh filename=package://meshes/schunk_left/f13.stl
- link Lmiddle_2: geometry collision mesh filename=package://meshes/schunk_left/f21.stl; visual mesh filename=package://meshes/schunk_left/f21.stl
- link Lmiddle_3: geometry collision mesh filename=package://meshes/schunk_left/f22.stl; visual mesh filename=package://meshes/schunk_left/f22.stl
- link Lmiddle_4: geometry collision mesh filename=package://meshes/schunk_left/f23.stl; visual mesh filename=package://meshes/schunk_left/f23.stl
- link Lpinky_2: geometry collision mesh filename=package://meshes/schunk_left/f41.stl; visual mesh filename=package://meshes/schunk_left/f41.stl
- link Lpinky_3: geometry collision mesh filename=package://meshes/schunk_left/f42.stl; visual mesh filename=package://meshes/schunk_left/f42.stl
- link Lpinky_4: geometry collision mesh filename=package://meshes/schunk_left/f43.stl; visual mesh filename=package://meshes/schunk_left/f43.stl
- link Lthumb_1: geometry collision mesh filename=package://meshes/schunk_left/d10.stl scale=1 -1 1; visual mesh filename=package://meshes/schunk_left/d10.stl scale=1 -1 1
- link Lthumb_3: geometry collision mesh filename=package://meshes/schunk_left/d11.stl scale=1 -1 -1; visual mesh filename=package://meshes/schunk_left/d11.stl scale=1 -1 -1
- link Lthumb_4: geometry collision mesh filename=package://meshes/schunk_left/d12.stl scale=1 -1 -1; visual mesh filename=package://meshes/schunk_left/d12.stl scale=1 -1 -1
- link Lthumb_5: geometry collision mesh filename=package://meshes/schunk_left/d13.stl scale=1 -1 -1; visual mesh filename=package://meshes/schunk_left/d13.stl scale=1 -1 -1
- link Lvirtual_index_1: geometry collision mesh filename=package://meshes/schunk_left/f10.stl; visual mesh filename=package://meshes/schunk_left/f10.stl
- link Lvirtual_middle_1: geometry collision mesh filename=package://meshes/schunk_left/f20.stl; visual mesh filename=package://meshes/schunk_left/f20.stl
- link Lvirtual_pinky_1: geometry collision mesh filename=package://meshes/schunk_left/f40.stl; visual mesh filename=package://meshes/schunk_left/f40.stl
- link left_hand_base: geometry collision mesh filename=package://meshes/schunk_left/base10.stl; visual mesh filename=package://meshes/schunk_left/base10.stl
- link ring_2: geometry collision mesh filename=package://meshes/schunk_left/f31.stl; visual mesh filename=package://meshes/schunk_left/f31.stl
- link ring_3: geometry collision mesh filename=package://meshes/schunk_left/f32.stl; visual mesh filename=package://meshes/schunk_left/f32.stl
- link ring_4: geometry collision mesh filename=package://meshes/schunk_left/f33.stl; visual mesh filename=package://meshes/schunk_left/f33.stl
- link virtual_ring_1: geometry collision mesh filename=package://meshes/schunk_left/f30.stl; visual mesh filename=package://meshes/schunk_left/f30.stl

File: yumi_gym/envs/assets/schunk_right_hand.urdf (robot description, URDF)
Before this commit: robot right_schunk_hand, 31 links, 30 joints
Links:
- link Re1: geometry collision mesh filename=package://meshes/schunk_right/H10.stl scale=1 1 1; visual mesh filename=package://meshes/schunk_right/H10.stl scale=1 1 1
- link Re2: geometry collision mesh filename=package://meshes/schunk_right/H11.stl scale=1 1 1; visual mesh filename=package://meshes/schunk_right/H11.stl scale=1 1 1
- link Rindex_2: geometry collision mesh filename=package://meshes/schunk_right/F11.stl; visual mesh filename=package://meshes/schunk_right/F11.stl
- link Rindex_3: geometry collision mesh filename=package://meshes/schunk_right/F12.stl; visual mesh filename=package://meshes/schunk_right/F12.stl
- link Rindex_4: geometry collision mesh filename=package://meshes/schunk_right/F13.stl; visual mesh filename=package://meshes/schunk_right/F13.stl
- link Rmiddle_2: geometry collision mesh filename=package://meshes/schunk_right/F21.stl; visual mesh filename=package://meshes/schunk_right/F21.stl
- link Rmiddle_3: geometry collision mesh filename=package://meshes/schunk_right/F22.stl; visual mesh filename=package://meshes/schunk_right/F22.stl
- link Rmiddle_4: geometry collision mesh filename=package://meshes/schunk_right/F23.stl; visual mesh filename=package://meshes/schunk_right/F23.stl
- link Rpinky_2: geometry collision mesh filename=package://meshes/schunk_right/F41.stl; visual mesh filename=package://meshes/schunk_right/F41.stl
- link Rpinky_3: geometry collision mesh filename=package://meshes/schunk_right/F42.stl; visual mesh filename=package://meshes/schunk_right/F42.stl
- link Rpinky_4: geometry collision mesh filename=package://meshes/schunk_right/F43.stl; visual mesh filename=package://meshes/schunk_right/F43.stl
- link Rring_2: geometry collision mesh filename=package://meshes/schunk_right/F31.stl; visual mesh filename=package://meshes/schunk_right/F31.stl
- link Rring_3: geometry collision mesh filename=package://meshes/schunk_right/F32.stl; visual mesh filename=package://meshes/schunk_right/F32.stl
- link Rring_4: geometry collision mesh filename=package://meshes/schunk_right/F33.stl; visual mesh filename=package://meshes/schunk_right/F33.stl
- link Rthumb_1: geometry collision mesh filename=package://meshes/schunk_right/D10.stl scale=1 1 1; visual mesh filename=package://meshes/schunk_right/D10.stl scale=1 1 1
- link Rthumb_3: geometry collision mesh filename=package://meshes/schunk_right/D11.stl scale=1 1 1; visual mesh filename=package://meshes/schunk_right/D11.stl scale=1 1 1
- link Rthumb_4: geometry collision mesh filename=package://meshes/schunk_right/D12.stl scale=1 1 1; visual mesh filename=package://meshes/schunk_right/D12.stl scale=1 1 1
- link Rthumb_5: geometry collision mesh filename=package://meshes/schunk_right/D13.stl scale=1 1 1; visual mesh filename=package://meshes/schunk_right/D13.stl scale=1 1 1
- link Rvirtual_index_1: geometry collision mesh filename=package://meshes/schunk_right/F10.stl; visual mesh filename=package://meshes/schunk_right/F10.stl
- link Rvirtual_middle_1: geometry collision mesh filename=package://meshes/schunk_right/F20.stl; visual mesh filename=package://meshes/schunk_right/F20.stl
- link Rvirtual_pinky_1: geometry collision mesh filename=package://meshes/schunk_right/F40.stl; visual mesh filename=package://meshes/schunk_right/F40.stl
- link Rvirtual_ring_1: geometry collision mesh filename=package://meshes/schunk_right/F30.stl; visual mesh filename=package://meshes/schunk_right/F30.stl
- link right_hand_base: geometry collision mesh filename=package://meshes/schunk_right/Base10.stl; visual mesh filename=package://meshes/schunk_right/Base10.stl

File: yumi_gym/envs/assets/yumi_arm.urdf (robot description, URDF)
Before this commit: robot yumi, 17 links, 16 joints
Links:
- link yumi_body: geometry collision mesh filename=package://meshes/coarse/body.stl; visual mesh filename=package://meshes/body.stl

File: yumi_gym/envs/assets/yumi_with_schunk_hands.urdf (robot description, URDF)
Before this commit: robot yumi, 79 links, 78 joints
Links:
- link Le1: geometry collision mesh filename=package://meshes/schunk_left/h10.stl scale=-1 1 1; visual mesh filename=package://meshes/schunk_left/h10.stl scale=-1 1 1
- link Le2: geometry collision mesh filename=package://meshes/schunk_left/h11.stl scale=-1 1 1; visual mesh filename=package://meshes/schunk_left/h11.stl scale=-1 1 1
- link Lindex_2: geometry collision mesh filename=package://meshes/schunk_left/f11.stl; visual mesh filename=package://meshes/schunk_left/f11.stl
- link Lindex_3: geometry collision mesh filename=package://meshes/schunk_left/f12.stl; visual mesh filename=package://meshes/schunk_left/f12.stl
- link Lindex_4: geometry collision mesh filename=package://meshes/schunk_left/f13.stl; visual mesh filename=package://meshes/schunk_left/f13.stl
- link Lmiddle_2: geometry collision mesh filename=package://meshes/schunk_left/f21.stl; visual mesh filename=package://meshes/schunk_left/f21.stl
- link Lmiddle_3: geometry collision mesh filename=package://meshes/schunk_left/f22.stl; visual mesh filename=package://meshes/schunk_left/f22.stl
- link Lmiddle_4: geometry collision mesh filename=package://meshes/schunk_left/f23.stl; visual mesh filename=package://meshes/schunk_left/f23.stl
- link Lpinky_2: geometry collision mesh filename=package://meshes/schunk_left/f41.stl; visual mesh filename=package://meshes/schunk_left/f41.stl
- link Lpinky_3: geometry collision mesh filename=package://meshes/schunk_left/f42.stl; visual mesh filename=package://meshes/schunk_left/f42.stl
- link Lpinky_4: geometry collision mesh filename=package://meshes/schunk_left/f43.stl; visual mesh filename=package://meshes/schunk_left/f43.stl
- link Lthumb_1: geometry collision mesh filename=package://meshes/schunk_left/d10.stl scale=1 -1 1; visual mesh filename=package://meshes/schunk_left/d10.stl scale=1 -1 1
- link Lthumb_3: geometry collision mesh filename=package://meshes/schunk_left/d11.stl scale=1 -1 -1; visual mesh filename=package://meshes/schunk_left/d11.stl scale=1 -1 -1
- link Lthumb_4: geometry collision mesh filename=package://meshes/schunk_left/d12.stl scale=1 -1 -1; visual mesh filename=package://meshes/schunk_left/d12.stl scale=1 -1 -1
- link Lthumb_5: geometry collision mesh filename=package://meshes/schunk_left/d13.stl scale=1 -1 -1; visual mesh filename=package://meshes/schunk_left/d13.stl scale=1 -1 -1
- link Lvirtual_index_1: geometry collision mesh filename=package://meshes/schunk_left/f10.stl; visual mesh filename=package://meshes/schunk_left/f10.stl
- link Lvirtual_middle_1: geometry collision mesh filename=package://meshes/schunk_left/f20.stl; visual mesh filename=package://meshes/schunk_left/f20.stl
- link Lvirtual_pinky_1: geometry collision mesh filename=package://meshes/schunk_left/f40.stl; visual mesh filename=package://meshes/schunk_left/f40.stl
- link Re1: geometry collision mesh filename=package://meshes/schunk_right/H10.stl scale=1 1 1; visual mesh filename=package://meshes/schunk_right/H10.stl scale=1 1 1
- link Re2: geometry collision mesh filename=package://meshes/schunk_right/H11.stl scale=1 1 1; visual mesh filename=package://meshes/schunk_right/H11.stl scale=1 1 1
- link Rindex_2: geometry collision mesh filename=package://meshes/schunk_right/F11.stl; visual mesh filename=package://meshes/schunk_right/F11.stl
- link Rindex_3: geometry collision mesh filename=package://meshes/schunk_right/F12.stl; visual mesh filename=package://meshes/schunk_right/F12.stl
- link Rindex_4: geometry collision mesh filename=package://meshes/schunk_right/F13.stl; visual mesh filename=package://meshes/schunk_right/F13.stl
- link Rmiddle_2: geometry collision mesh filename=package://meshes/schunk_right/F21.stl; visual mesh filename=package://meshes/schunk_right/F21.stl
- link Rmiddle_3: geometry collision mesh filename=package://meshes/schunk_right/F22.stl; visual mesh filename=package://meshes/schunk_right/F22.stl
- link Rmiddle_4: geometry collision mesh filename=package://meshes/schunk_right/F23.stl; visual mesh filename=package://meshes/schunk_right/F23.stl
- link Rpinky_2: geometry collision mesh filename=package://meshes/schunk_right/F41.stl; visual mesh filename=package://meshes/schunk_right/F41.stl
- link Rpinky_3: geometry collision mesh filename=package://meshes/schunk_right/F42.stl; visual mesh filename=package://meshes/schunk_right/F42.stl
- link Rpinky_4: geometry collision mesh filename=package://meshes/schunk_right/F43.stl; visual mesh filename=package://meshes/schunk_right/F43.stl
- link Rring_2: geometry collision mesh filename=package://meshes/schunk_right/F31.stl; visual mesh filename=package://meshes/schunk_right/F31.stl
- link Rring_3: geometry collision mesh filename=package://meshes/schunk_right/F32.stl; visual mesh filename=package://meshes/schunk_right/F32.stl
- link Rring_4: geometry collision mesh filename=package://meshes/schunk_right/F33.stl; visual mesh filename=package://meshes/schunk_right/F33.stl
- link Rthumb_1: geometry collision mesh filename=package://meshes/schunk_right/D10.stl scale=1 1 1; visual mesh filename=package://meshes/schunk_right/D10.stl scale=1 1 1
- link Rthumb_3: geometry collision mesh filename=package://meshes/schunk_right/D11.stl scale=1 1 1; visual mesh filename=package://meshes/schunk_right/D11.stl scale=1 1 1
- link Rthumb_4: geometry collision mesh filename=package://meshes/schunk_right/D12.stl scale=1 1 1; visual mesh filename=package://meshes/schunk_right/D12.stl scale=1 1 1
- link Rthumb_5: geometry collision mesh filename=package://meshes/schunk_right/D13.stl scale=1 1 1; visual mesh filename=package://meshes/schunk_right/D13.stl scale=1 1 1
- link Rvirtual_index_1: geometry collision mesh filename=package://meshes/schunk_right/F10.stl; visual mesh filename=package://meshes/schunk_right/F10.stl
- link Rvirtual_middle_1: geometry collision mesh filename=package://meshes/schunk_right/F20.stl; visual mesh filename=package://meshes/schunk_right/F20.stl
- link Rvirtual_pinky_1: geometry collision mesh filename=package://meshes/schunk_right/F40.stl; visual mesh filename=package://meshes/schunk_right/F40.stl
- link Rvirtual_ring_1: geometry collision mesh filename=package://meshes/schunk_right/F30.stl; visual mesh filename=package://meshes/schunk_right/F30.stl
- link left_hand_base: geometry collision mesh filename=package://meshes/schunk_left/base10.stl; visual mesh filename=package://meshes/schunk_left/base10.stl
- link right_hand_base: geometry collision mesh filename=package://meshes/schunk_right/Base10.stl; visual mesh filename=package://meshes/schunk_right/Base10.stl
- link ring_2: geometry collision mesh filename=package://meshes/schunk_left/f31.stl; visual mesh filename=package://meshes/schunk_left/f31.stl
- link ring_3: geometry collision mesh filename=package://meshes/schunk_left/f32.stl; visual mesh filename=package://meshes/schunk_left/f32.stl
- link ring_4: geometry collision mesh filename=package://meshes/schunk_left/f33.stl; visual mesh filename=package://meshes/schunk_left/f33.stl
- link virtual_ring_1: geometry collision mesh filename=package://meshes/schunk_left/f30.stl; visual mesh filename=package://meshes/schunk_left/f30.stl

Commit message: see collision

File: yumi_gym/envs/assets/schunk_left_hand.urdf (robot description, URDF)
Before this commit: robot left_schunk_hand, 31 links, 30 joints
Links:
- removed link ring_2
- removed link ring_3
- removed link ring_4
- removed link virtual_ring_1
- added link Lring_2; collision mesh filename=package://meshes/schunk_left/f31.stl; visual mesh filename=package://meshes/schunk_left/f31.stl
- added link Lring_3; collision mesh filename=package://meshes/schunk_left/f32.stl; visual mesh filename=package://meshes/schunk_left/f32.stl
- added link Lring_4; collision mesh filename=package://meshes/schunk_left/f33.stl; visual mesh filename=package://meshes/schunk_left/f33.stl
- added link Lvirtual_ring_1; collision mesh filename=package://meshes/schunk_left/f30.stl; visual mesh filename=package://meshes/schunk_left/f30.stl
Joints:
- joint LRing_3: child ring_3 -> Lring_3; parent ring_2 -> Lring_2
- joint LRing_4: child ring_4 -> Lring_4; parent ring_3 -> Lring_3
- joint LRing_Proximal: child ring_2 -> Lring_2; parent virtual_ring_1 -> Lvirtual_ring_1
- joint LRing_Spread: child virtual_ring_1 -> Lvirtual_ring_1

File: yumi_gym/envs/assets/yumi_with_schunk_hands.urdf (robot description, URDF)
Before this commit: robot yumi, 79 links, 78 joints
Links:
- removed link ring_2
- removed link ring_3
- removed link ring_4
- removed link virtual_ring_1
- added link Lring_2; collision mesh filename=package://meshes/schunk_left/f31.stl; visual mesh filename=package://meshes/schunk_left/f31.stl
- added link Lring_3; collision mesh filename=package://meshes/schunk_left/f32.stl; visual mesh filename=package://meshes/schunk_left/f32.stl
- added link Lring_4; collision mesh filename=package://meshes/schunk_left/f33.stl; visual mesh filename=package://meshes/schunk_left/f33.stl
- added link Lvirtual_ring_1; collision mesh filename=package://meshes/schunk_left/f30.stl; visual mesh filename=package://meshes/schunk_left/f30.stl
Joints:
- joint LRing_3: child ring_3 -> Lring_3; parent ring_2 -> Lring_2
- joint LRing_4: child ring_4 -> Lring_4; parent ring_3 -> Lring_3
- joint LRing_Proximal: child ring_2 -> Lring_2; parent virtual_ring_1 -> Lvirtual_ring_1
- joint LRing_Spread: child virtual_ring_1 -> Lvirtual_ring_1
